Commit message: update urdf based on the real robot setup

File: assets/franka_panda/panda.urdf (robot description, URDF)
Before this commit: robot Panda, 13 links, 12 joints
Joints:
- joint panda_wrist_hand: origin xyz=-0.03 -0.03 0.02 rpy=0 0 2.356109 -> xyz=0.070688 0.100659 0.041000 rpy=0.477868 0.002474 -0.799077

Commit message: corrected wirst camera position

File: assets/franka_panda/panda.urdf (robot description, URDF)
Before this commit: robot Panda, 13 links, 12 joints
Joints:
- joint panda_wrist_hand: origin xyz=0.070688 0.100659 0.041000 rpy=0.477868 0.002474 -0.799077 -> xyz=0.070688 0.100659 -0.003400 rpy=0.477868 0.002474 -0.799077
